Commit message: Add ore spawning during mining

File: bugger_description/urdf/bugger.urdf (robot description, URDF)
Before this commit: robot simple_robot, 10 links, 9 joints
Links:
- added link ore_spawn_point
- link container: geometry collision box size=0.01 0.26 0.1; collision box size=0.01 0.26 0.18
Joints:
- added joint ore_spawn_point_joint: type fixed, parent container, child ore_spawn_point, origin xyz=0.2 0 0.2 rpy=0 0 0, axis 0 0 0
