Commit message: Add auto-dumping feature
- Add two drop off sensors in the back of bagger

- Create dumping_executor node to control the dumping sequence

File: bagger_description/urdf/bagger.urdf (robot description, URDF)
Before this commit: robot simple_robot, 11 links, 10 joints
Links:
- added link left_right_ground_distance_sensor_link; visual box size=0.02 0.02 0.02
- added link rear_right_ground_distance_sensor_link; visual box size=0.02 0.02 0.02
Joints:
- added joint left_right_ground_distance_sensor_joint: type fixed, parent chassis, child left_right_ground_distance_sensor_link, origin xyz=-0.265 0.16 0.01 rpy=0 0 0
- added joint rear_right_ground_distance_sensor_joint: type fixed, parent chassis, child rear_right_ground_distance_sensor_link, origin xyz=-0.265 -0.16 0.01 rpy=0 0 0

Commit message: Change coordinate transformation in ore_spawner.py with only TFMessage, no tf2_ros
I thought it would significantly reduce complexity :)

File: bagger_description/urdf/bagger.urdf (robot description, URDF)
Before this commit: robot simple_robot, 13 links, 12 joints
Links:
- removed link ore_spawn_point
- added link ore_collection_point, mass 0.001
Joints:
- removed joint ore_spawn_point_joint
- added joint ore_collection_point_joint: type fixed, parent container, child ore_collection_point, origin xyz=0.2 0 0.2 rpy=0 0 0, axis 0 0 0

Commit message: Update heap spawning, ore collection point, and PID parameters
- Replace generate_heaps.py and heaps.sdf with spawn_heaps.launch.py (cannot teleport child models in nested models)
- Adjust ore_collection_point position to prevent overlapping cubes
- Update PID bucket wheel parameters (unwinding and i_max/i_min issues persist)
- Refactor ore_spawner.py variable names

File: bagger_description/urdf/bagger.urdf (robot description, URDF)
Before this commit: robot simple_robot, 13 links, 12 joints
Joints:
- joint ore_collection_point_joint: origin xyz=0.2 0 0.2 rpy=0 0 0 -> xyz=0.2 0 0.4 rpy=0 0 0

Commit message: feat(control): add bucket wheel PID controller and refactor launch setup
- Add PID controller configuration for bucket wheel
- Switch bucket wheel velocity interface from Float64 to MultiDOFCommand
- Update controller manager to publish joint states
- Add bagger_sim.urdf.xacro (top-level) and bagger.gazebo.xacro (PID topic remapping) to bagger_gazebo
- Move robot_state_publisher to gazebo.launch.py
- Move contact plugin configuration to warehouse_world.sdf

File: bagger_description/urdf/bagger.urdf (robot description, URDF)
Before this commit: robot simple_robot, 13 links, 12 joints
Joints:
- joint bucket_wheel_joint: limit effort=100.0 velocity=1.0 -> effort=100.0 velocity=10.0

Commit message: WIP

File: bagger_description/urdf/bagger.urdf (robot description, URDF)
Before this commit: robot bagger, 13 links, 12 joints
Links:
- added link camera_mast_link; visual box size=0.03 0.03 0.03
Joints:
- added joint camera_mast_joint: type fixed, parent chassis, child camera_mast_link, origin xyz=0.3 0.0 0.45 rpy=0 0.436 0

Commit message: feat: align arm to cube height and correct camera TF
- Add arm alignment after navigation with TF freshness and reachability checks.
- Remove PoseStamped topic publication; publish detected cube poses only through TF, using cube names as frame IDs.
- Expand teleop arm limits to +/-0.75 rad.

OpenCV returns coordinates using optical axes: X right, Y down, Z forward. Previously, these values were labelled with camera_mast_link, whose axes are X forward, Y left, Z up. TF interpreted the numbers along the wrong axes, producing incorrect cube heights in map.

Add camera_optical_frame with a fixed rotation and use that name in camera headers. This lets TF apply the missing rotation when converting cube poses into map.

File: bagger_description/urdf/bagger.urdf (robot description, URDF)
Before this commit: robot bagger, 14 links, 13 joints
Links:
- added link camera_optical_frame
Joints:
- added joint camera_optical_joint: type fixed, parent camera_mast_link, child camera_optical_frame, origin xyz=0 0 0 rpy=-1.5707963267948966 0 -1.5707963267948966

Commit message: feat: add autonomous cube collection and container weight sensing
- Align with the cube using TF, drive toward it, and spin the bucket wheel through the existing controller.
- Add and bridge a container force/torque sensor to estimate the contents' weight and cube count.
- Stop driving and spinning the wheel once stable weight readings confirm a load.
- Level the caster mounting and reduce spawning and collection delays.
- Remove unused cube pose publishers from perception

File: bagger_description/urdf/bagger.urdf (robot description, URDF)
Before this commit: robot bagger, 15 links, 14 joints
Joints:
- joint caster_wheel_joint: origin xyz=0.2 0 0.002 -> xyz=0.2 0 0.000

Commit message: feat: add dumping to autonomy sequence, tune unloading, and raise lidar

File: bagger_description/urdf/bagger.urdf (robot description, URDF)
Before this commit: robot bagger, 15 links, 14 joints
Joints:
- joint container_joint: limit lower=-1.75 upper=0 effort=100.0 velocity=0.5 -> lower=-2.9 upper=0 effort=200.0 velocity=0.5
- joint lidar_joint: origin xyz=0.2 0 0.37 rpy=0 0 0 -> xyz=0.2 0 0.65 rpy=0 0 0
